File: hardware/USB-Weather.brd (EAGLE design)
At the start: 50.8 x 66 mm, 74 parts, among them U1 ATMEGA328, U2 MIC5219-3.3BM5, U3 FT232RL, U5 HTU21DSMD, U6 TEMT6000, U7 BMP180, Y1 8MHz

Commit message: revision in progress
Parts:
- removed U3: FT232RL, SparkFun:SSOP28DB
- added C13, C14: 4.7uF, SparkFun:0603-CAP
- added C15: 0.1uF, SparkFun:0603-CAP
- added D12: RED, SparkFun:LED-0603
- added JP10: 1X2, SparkFun:1X02_NO_SILK
- added JP9: (no value), mike-temp:1X02_NO_SILK
- added R18: 330, SparkFun:0603-RES
- added R19: 2K, SparkFun:0603-RES
- added R20: (no value), SparkFun:1/6W-RES
- added R21, R22: 27, SparkFun:0603-RES
- added U4: MCP73831, SparkFun:SOT23-5
- added U8: FT231XS, mike-temp:SSOP20_L
- JP6: device mike-temp:1X04_NO_SILK_ROUND -> mike-temp:1X03_ROUND_ONLY_NO_SILK
- moved JP6 33.0 mm to (20.3, 29.2)
- moved JP5 21.6 mm to (38.1, 34.3)
- moved C8 12.2 mm to (13.7, 6.99), turned to 180 degrees
- moved LOGO1 11.4 mm to (1.27, 61.0)
- moved U$1 5.08 mm to (25.1, -3.43)
- moved R3 4.02 mm to (17.1, 22.9), turned to 180 degrees
- moved JP3 2.84 mm to (25.4, 26.7)
- moved C5 1.27 mm to (16.5, 18.4)
- moved C6 1.27 mm to (26.7, 17.1)
- moved C7 1.27 mm to (26.7, 19.7)
- moved U2 1.27 mm to (20.3, 18.4)
Connections:
- new net N$22: D12.A, R18.1
- new net N$23: JP4.D-, R21.2
- new net N$24: JP4.D+, R22.2
- new net PROG: R19.1, R20.1, U4.5
- new net STAT: D12.C, U4.1
- net 3V-INT: now also U8.13, U8.14, U8.3; no longer U3.17, U3.4
- net GND: now also C13.2, C14.2, C15.2, JP10.2, R19.2, R20.2, U4.2, U8.16, U8.6; no longer R7.2, U3.18, U3.21, U3.25, U3.26, U3.7
- net N$20: now also R7.2; no longer JP6.4
- net RX: now also JP9.1
- net TX: now also JP9.2, U8.4; no longer U3.5
- net USB-DTR: now also U8.1; no longer U3.2
- net USB-RX: now also U8.20; no longer U3.1
- net USB_D+: now also R22.1, U8.11; no longer JP4.D+, U3.15
- net USB_D-: now also R21.1, U8.12; no longer JP4.D-, U3.16
- net VBAT: now also C14.1, U4.3
- net VUSB: now also C13.1, C15.1, JP10.1, R18.2, U4.4, U8.15; no longer U3.20
Routing:
- net 3V-INT: track 29.8 -> 4.17 mm
- net N$17: track 0.00 -> 25.6 mm, vias 0 -> 1
- net N$16: track 0.00 -> 22.0 mm, vias 0 -> 1
- net N$15: track 0.00 -> 19.1 mm, vias 0 -> 1
- net N$20: track 0.00 -> 11.7 mm, vias 0 -> 2
- net MOSI: track 6.62 -> 16.6 mm
- net VCC: track 315.3 -> 306.9 mm
- net RF-CTS: track 58.2 -> 49.9 mm
- net RX: track 29.4 -> 36.5 mm
- net MISO: track 3.75 -> 9.42 mm
- net VRAW: track 51.2 -> 46.3 mm
- net USB_D+: track 8.91 -> 4.48 mm
- net N$6: track 4.33 -> 0.00 mm
- net N$19: track 0.00 -> 4.21 mm
- net N$21: track 0.00 -> 3.88 mm
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Other:
- board text added: "Charge"

Commit message: pre-review
Parts:
- removed C13: 4.7uF, SparkFun:0603-CAP
- removed U$1: LOGO-SFENEW, SparkFun:SFE-NEW-WEBLOGO
- added D13: BAS16, SparkFun:SOD-323
- added LOGO2: OSHW-LOGOS, SparkFun-Aesthetics:OSHW-LOGO-S
- added LOGO3: SFE_LOGO_NAME.1_INCH, SparkFun-Aesthetics:SFE_LOGO_NAME_.1
- added R23: 10K, SparkFun:0603-RES
- D12: value RED -> YELLOW
- JP8: device SparkFun:1X02 -> mike-temp:1X02_NO_SILK
- LOGO1: value OSHW_LOGO_FILLX0100-NT -> LOGO-SFENEW; device OSHW:OSHW_FILLX100_NOTEXT -> SparkFun-Aesthetics:SFE-NEW-WEBLOGO
- moved LOGO1 68.8 mm to (35.6, 1.27), flipped to the bottom, turned to 0 degrees
- moved JP10 14.5 mm to (11.4, 10.2), turned to 90 degrees
- moved C15 10.8 mm to (28.6, 6.99)
- moved D1 10.5 mm to (11.1, 3.81)
- moved R1 10.5 mm to (7.94, 3.81)
- moved C14 8.25 mm to (32.4, 11.4)
- moved D2 7.30 mm to (20.0, 3.81)
- moved R2 7.30 mm to (16.8, 3.81)
- moved R19 4.45 mm to (24.8, 11.4)
- moved R20 4.45 mm to (24.8, 11.4)
- moved R21 3.51 mm to (13.7, 13.0)
- moved R22 3.51 mm to (13.7, 9.84), turned to 270 degrees
- moved C8 3.24 mm to (16.8, 6.35)
- moved U8 3.18 mm to (19.1, 11.4)
- moved U4 1.90 mm to (28.6, 11.4), turned to 90 degrees
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Connections:
- net 3V-INT renamed N$26
- net N$15 renamed A1
- net N$16 renamed A2
- net N$17 renamed A3
- net N$18 renamed D8
- net N$19 renamed D9
- net N$20 renamed BATT_GND
- net N$21 renamed D7
- removed net N$4: R2.2, U1.2
- new net N$25: D13.2, JP4.VBUS, U8.15
- new net XSLEEP: JP6-DNP.9, R23.2, U1.2
- net GND: now also JP10.1; no longer C13.2, JP10.2
- net MOSI: now also R2.2
- net VBAT: now also S1.1; no longer S1.3
- net VCC: now also R23.1
- net VUSB: now also D13.1, JP10.2; no longer C13.1, JP10.1, JP4.VBUS, S1.1, U8.15
Routing:
- net N$4: track 81.7 -> 0.00 mm, vias 2 -> 0
- net MOSI: track 16.6 -> 65.3 mm, vias 0 -> 2
- net XSLEEP: track 0.00 -> 33.9 mm, vias 0 -> 2
- net VCC: track 306.9 -> 328.3 mm, vias 6 -> 7
- net N$25: track 0.00 -> 19.1 mm
- net N$26: track 4.17 -> 19.7 mm
- net VBAT: track 58.5 -> 69.6 mm, vias 2 -> 3
- net STAT: track 0.00 -> 8.82 mm
- net N$24: track 3.00 -> 8.79 mm
- net VRAW: track 46.3 -> 51.4 mm
- net N$6: track 0.00 -> 4.73 mm
- net PROG: track 0.00 -> 4.26 mm
- net N$23: track 2.83 -> 6.64 mm
- net VUSB: track 35.4 -> 32.3 mm, vias 0 -> 1
- net TX: track 103.0 -> 105.8 mm
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Other:
- board text added: "33"
- board text added: "A1"
- board text added: "A2"
- board text added: "A3"
- board text added: "CHG"
- board text added: "D7"
- board text added: "D8"
- board text added: "D9"
- board text added: "GD"
- board text added: "RX"
- board text added: "TX"
- board text added: "V4"
- board text added: "Weather"
- board text removed: "USB Weather V4"

Commit message: Minor updates for reveiw
Parts:
- JP3: device SparkFun:2X3 -> mike-temp:2X3
- moved R23 0.71 mm to (4.76, 59.1)
- moved D13 0.64 mm to (11.4, 16.5)
- moved LOGO2 0.64 mm to (1.91, 59.7)
- moved R21 0.32 mm to (13.7, 13.3)
- moved R22 0.32 mm to (13.7, 9.53)
Routing:
- net N$25: track 19.1 -> 20.8 mm
- net VCC: track 328.3 -> 329.3 mm
- net VUSB: track 32.3 -> 33.0 mm
Other:
- board text added: "4.2-6V"
- board text added: "CHARGE"
- board text added: "OFF"
- board text added: "ON"
- board text removed: "CHG"
