File: hardware/USB-Weather.sch (EAGLE design)
At the start: 72 parts, among them U1 ATMEGA328, U2 MIC5219-3.3BM5, U3 FT232RL, U5 HTU21DSMD, U6 TEMT6000, U7 BMP180, Y1 8MHz

Commit message: revision in progress
Parts:
- removed U3: FT232RL, SparkFun:FT232RL-BASICSSOP
- added C13, C14: 4.7uF, SparkFun:CAP0603-CAP
- added C15: 0.1uF, SparkFun:CAP0603-CAP
- added D12: RED, SparkFun:LED0603
- added JP10: 1X2, SparkFun:M021X02_NO_SILK
- added JP9: (no value), mike-temp:M021X02_NO_SILK
- added R18: 330, SparkFun:RESISTOR0603-RES
- added R19: 2K, SparkFun:RESISTOR0603-RES
- added R20: (no value), SparkFun:RESISTORPTH-1/6W
- added R21, R22: 27, SparkFun:RESISTOR0603-RES
- added U4: MCP73831, SparkFun:MCP73831
- added U8: FT231XS, mike-temp:FT231XS
- JP6: device mike-temp:M041X04_NO_SILK_ROUND -> mike-temp:M03_ROUND_ONLY_NO_SILK
Connections:
- new net N$22: D12.A, R18.1
- new net N$23: JP4.D-, R21.2
- new net N$24: JP4.D+, R22.2
- new net PROG: R19.1, R20.1, U4.PROG
- new net STAT: D12.C, U4.STAT
- net 3V-INT: now also U8.!RESET, U8.3V3OUT, U8.VCCIO; no longer U3.3V3OUT, U3.VCCIO
- net GND: now also C13.2, C14.2, C15.2, JP10.2, R19.2, R20.2, U4.VSS, U8.GND@16, U8.GND@6; no longer R7.2, U3.AGND, U3.GND1, U3.GND2, U3.GND3, U3.TEST
- net N$20: now also R7.2; no longer JP6.4
- net RX: now also JP9.1
- net TX: now also JP9.2, U8.RXD; no longer U3.RXD
- net USB-DTR: now also U8.!DTR; no longer U3.DTR
- net USB-RX: now also U8.TXD; no longer U3.TXD
- net USB_D+: now also R22.1, U8.USBDP; no longer JP4.D+, U3.USBDP
- net USB_D-: now also R21.1, U8.USBDM; no longer JP4.D-, U3.USBDM
- net VBAT: now also C14.1, U4.VBAT
- net VUSB: now also C13.1, C15.1, JP10.1, R18.2, U4.VIN, U8.VCC; no longer U3.VCC
Other:
- note added: "Set for 500mA charging"
- moved on the sheet: C8, D2, R2

Commit message: pre-review
Parts:
- removed C13: 4.7uF, SparkFun:CAP0603-CAP
- removed U$1: LOGO-SFENEW, SparkFun:LOGO-SFENEW
- added D13: BAS16, SparkFun:DIODESOD
- added LOGO2: OSHW-LOGOS, SparkFun-Aesthetics:OSHW-LOGOS
- added LOGO3: SFE_LOGO_NAME.1_INCH, SparkFun-Aesthetics:SFE_LOGO_NAME.1_INCH
- added R23: 10K, SparkFun:RESISTOR0603-RES
- D12: value RED -> YELLOW
- JP8: device SparkFun:M02PTH -> mike-temp:M021X02_NO_SILK
- LOGO1: value OSHW_LOGO_FILLX0100-NT -> LOGO-SFENEW; device OSHW:OSHW_LOGO_FILLX0100-NT -> SparkFun-Aesthetics:LOGO-SFENEW
Connections:
- net 3V-INT renamed N$26
- net N$15 renamed A1
- net N$16 renamed A2
- net N$17 renamed A3
- net N$18 renamed D8
- net N$19 renamed D9
- net N$20 renamed BATT_GND
- net N$21 renamed D7
- removed net N$4: R2.2, U1.PD4(XCK/T0)
- new net N$25: D13.A, JP4.VBUS, U8.VCC
- new net XSLEEP: JP6-DNP.DTR, R23.2, U1.PD4(XCK/T0)
- net GND: now also JP10.1; no longer C13.2, JP10.2
- net MOSI: now also R2.2
- net VBAT: now also S1.O; no longer S1.S
- net VCC: now also R23.1
- net VUSB: now also D13.C, JP10.2; no longer C13.1, JP10.1, JP4.VBUS, S1.O, U8.VCC
Other:
- note added: "A1"
- note added: "A2"
- note added: "A3"
- note added: "CHARGE"
- note added: "D10"
- note added: "D7"
- note added: "Lipo Charger"
- note added: "Pressure"
- note added: "V4 changes: BMP085 to BMP180 SHT15 to HTU21D added Lipo charger added Xbee sleep to D4 added battery voltage divider base to D9 moved status LED to D11"
- note removed: "*"
- note removed: "D11"
- note removed: "Power switch selects either"
- note removed: "Pressure*"
- note removed: "R. Owens, M. Grusin"
- note removed: "V3 changes SCP1000 pressure sensor to BMP085,"
- note removed: "V4 changes: BMP085 to BMP180 SHT15 to HTU21D"
- note removed: "adds header for XBee radio module"
- note removed: "adds inputs for SEN-08942 weather meters,"
- moved on the sheet: C1, C12, C14, C15, C2, C3, C4, C5, C6, C7, C8, D1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

Commit message: Minor updates for reveiw
Parts:
- JP3: device SparkFun:AVR_SPI_PRG_6PTH -> mike-temp:AVR_SPI_PRG_6PTH
Other:
- note added: "I2C address (7-bit): 0x40"
- note removed: "I2C address (3-bit): B000 (see datasheet)"
- moved on the sheet: R6, R7
Changed lines of the file:
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@@
 <?xml version="1.0" encoding="utf-8"?>
 <!DOCTYPE eagle SYSTEM "eagle.dtd">
-<eagle version="6.4">
+<eagle version="6.5.0">
 <drawing>
 <settings>
@@
 <part name="U$4" library="SparkFun" deviceset="STAND-OFF" device=""/>
 <part name="U$5" library="SparkFun" deviceset="STAND-OFF" device=""/>
-<part name="JP3" library="SparkFun" deviceset="AVR_SPI_PRG_6" device="PTH" value="AVR_Prog"/>
+<part name="JP3" library="mike-temp" deviceset="AVR_SPI_PRG_6" device="PTH" value="AVR_Prog"/>
 <part name="GND30" library="SparkFun" deviceset="GND" device=""/>
 <part name="P+6" library="SparkFun" deviceset="VCC" device=""/>
@@
 <text x="210.82" y="119.38" size="1.778" layer="95">Expansion connectors</text>
 <text x="73.66" y="134.62" size="1.778" layer="95">I2C address (7-bit): 0x77</text>
-<text x="2.54" y="134.62" size="1.778" layer="95">I2C address (3-bit): B000 (see datasheet)</text>
+<text x="2.54" y="134.62" size="1.778" layer="95">I2C address (7-bit): 0x40</text>
 <text x="17.78" y="58.42" size="1.778" layer="95">ISP programming header</text>
 <text x="139.7" y="101.6" size="1.778" layer="94">A0</text>
@@
 </instance>
 <instance part="GND27" gate="1" x="63.5" y="76.2"/>
-<instance part="R7" gate="G$1" x="187.96" y="76.2" rot="MR270"/>
-<instance part="R6" gate="G$1" x="187.96" y="93.98" rot="MR270"/>
+<instance part="R7" gate="G$1" x="187.96" y="78.74" rot="MR270"/>
+<instance part="R6" gate="G$1" x="187.96" y="99.06" rot="MR270"/>
 <instance part="U$2" gate="G$1" x="246.38" y="25.4"/>
 <instance part="U$3" gate="G$1" x="241.3" y="25.4"/>
@@
 <segment>
 <wire x1="137.16" y1="86.36" x2="187.96" y2="86.36" width="0.1524" layer="91"/>
-<wire x1="187.96" y1="86.36" x2="187.96" y2="88.9" width="0.1524" layer="91"/>
-<wire x1="187.96" y1="86.36" x2="187.96" y2="81.28" width="0.1524" layer="91"/>
+<wire x1="187.96" y1="86.36" x2="187.96" y2="93.98" width="0.1524" layer="91"/>
+<wire x1="187.96" y1="86.36" x2="187.96" y2="83.82" width="0.1524" layer="91"/>
 <junction x="187.96" y="86.36"/>
 <label x="147.32" y="86.36" size="1.778" layer="95"/>
@@
 <net name="VBAT" class="0">
 <segment>
-<wire x1="187.96" y1="99.06" x2="187.96" y2="116.84" width="0.1524" layer="91"/>
+<wire x1="187.96" y1="104.14" x2="187.96" y2="116.84" width="0.1524" layer="91"/>
 <label x="184.912" y="117.602" size="1.778" layer="95"/>
 <pinref part="R6" gate="G$1" pin="1"/>
@@
 <pinref part="U1" gate="G$1" pin="PB2(SS/OC1B)"/>
 <wire x1="137.16" y1="50.8" x2="187.96" y2="50.8" width="0.1524" layer="91"/>
-<wire x1="187.96" y1="50.8" x2="187.96" y2="71.12" width="0.1524" layer="91"/>
+<wire x1="187.96" y1="50.8" x2="187.96" y2="73.66" width="0.1524" layer="91"/>
 <label x="147.32" y="50.8" size="1.778" layer="95"/>
 </segment>
